File: pcb/SolarLoRaBox.kicad_pcb (KiCad board)
At the start: 4 copper layers, 71.3 x 92.8 mm, 57 parts, among them J1 Conn_01x02_Socket, J10 Conn_01x05_Socket, J2 Conn_01x02_Socket, J3 Conn_01x04_Socket, J4 Conn_ARM_SWD_TagConnect_TC2030, J5 Conn_01x04_Socket, J6 Conn_01x04_Socket, J7 Conn_01x04_Socket, J8 Conn_01x04_Socket, J9 Conn_01x04_Socket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

Commit message: pcb, sch: match silk print and schematic
Connections:
- net /GPIO1 renamed /GPIOD
- net /GPIO2 renamed /GPIOC
- net /GPIO3 renamed /GPIOB
- net /GPIO4 renamed /GPIOA
Changed lines of the file:
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@@
 	(net 53 "unconnected-(U7-DIO3-Pad8)")
 	(net 54 "Net-(J9-Pin_2)")
-	(net 55 "/GPIO1")
-	(net 56 "/GPIO3")
-	(net 57 "/GPIO2")
-	(net 58 "/GPIO4")
+	(net 55 "/GPIOA")
+	(net 56 "/GPIOD")
+	(net 57 "/GPIOB")
+	(net 58 "/GPIOC")
 	(footprint "Capacitor_SMD:C_0805_2012Metric_Pad1.18x1.45mm_HandSolder"
 		(layer "F.Cu")
@@
 			(layers "*.Cu" "*.Mask")
 			(remove_unused_layers no)
-			(net 58 "/GPIO4")
+			(net 55 "/GPIOA")
 			(pinfunction "Pin_2")
 			(pintype "passive")
@@
 			(layers "*.Cu" "*.Mask")
 			(remove_unused_layers no)
-			(net 56 "/GPIO3")
+			(net 57 "/GPIOB")
 			(pinfunction "Pin_3")
 			(pintype "passive")
@@
 			(layers "*.Cu" "*.Mask")
 			(remove_unused_layers no)
-			(net 57 "/GPIO2")
+			(net 58 "/GPIOC")
 			(pinfunction "Pin_4")
 			(pintype "passive")
@@
 			(layers "*.Cu" "*.Mask")
 			(remove_unused_layers no)
-			(net 55 "/GPIO1")
+			(net 56 "/GPIOD")
 			(pinfunction "Pin_5")
 			(pintype "passive")
@@
 			(layer "F.Fab")
 		)
-		(fp_text user "*"
-			(at -5.588 -3.381 0)
+		(fp_text user "${REFERENCE}"
+			(at 0 0 0)
+			(unlocked yes)
 			(layer "F.Fab")
 			(effects
@@
 			)
 		)
-		(fp_text user "${REFERENCE}"
-			(at 0 0 0)
-			(unlocked yes)
-			(layer "F.Fab")
-			(effects
-				(font
-					(size 1 1)
-					(thickness 0.15)
-				)
-			)
-		)
 		(pad "1" smd rect
 			(at -4.2164 -2.75 90)
@@
 			(size 0.2794 1.4732)
 			(layers "F.Cu" "F.Paste" "F.Mask")
-			(net 55 "/GPIO1")
+			(net 56 "/GPIOD")
 			(pinfunction "PB4")
 			(pintype "bidirectional")
@@
 			(size 0.2794 1.4732)
 			(layers "F.Cu" "F.Paste" "F.Mask")
-			(net 57 "/GPIO2")
+			(net 58 "/GPIOC")
 			(pinfunction "PB5")
 			(pintype "bidirectional")
@@
 			(size 0.2794 1.4732)
 			(layers "F.Cu" "F.Paste" "F.Mask")
-			(net 56 "/GPIO3")
+			(net 57 "/GPIOB")
 			(pinfunction "PB6")
 			(pintype "bidirectional")
@@
 			(size 0.2794 1.4732)
 			(layers "F.Cu" "F.Paste" "F.Mask")
-			(net 58 "/GPIO4")
+			(net 55 "/GPIOA")
 			(pinfunction "PB7")
 			(pintype "bidirectional")
@@
 			(pintype "power_in")
 		)
-		(model "${KICAD8_3DMODEL_DIR}/Package_DFN_QFN.3dshapes/TQFN-48-1EP_7x7mm_P0.5mm_EP5.1x5.1mm.wrl"
-			(offset
-				(xyz 0 0 0)
-			)
-			(scale
-				(xyz 1 1 1)
-			)
-			(rotate
-				(xyz 0 0 0)
-			)
-		)
-		(model "${KICAD8_3DMODEL_DIR}/Package_DFN_QFN.3dshapes/QFN-28-1EP_6x6mm_P0.65mm_EP4.25x4.25mm.step"
-			(offset
-				(xyz 0 0 0)
-			)
-			(scale
-				(xyz 1 1 1)
-			)
-			(rotate
-				(xyz 0 0 0)
-			)
-		)
-		(model "${KICAD8_3DMODEL_DIR}/Package_QFP.3dshapes/LQFP-48-1EP_7x7mm_P0.5mm_EP3.6x3.6mm.step"
-			(offset
-				(xyz 0 0 0)
-			)
-			(scale
-				(xyz 1 1 1)
-			)
-			(rotate
-				(xyz 0 0 0)
-			)
-		)
 	)
 	(footprint "Resistor_SMD:R_0805_2012Metric_Pad1.20x1.40mm_HandSolder"
@@
 	)
 	(segment
-		(start 245.57 35.79)
-		(end 247.38 35.79)
+		(start 243.15 36)
+		(end 243.15 35.97)
 		(width 0.3)
 		(layer "F.Cu")
@@
 	)
 	(segment
-		(start 227.52 59.8836)
-		(end 227.52 53.84)
+		(start 243.15 35.97)
+		(end 243.94 35.18)
 		(width 0.3)
 		(layer "F.Cu")
@@
 	)
 	(segment
-		(start 247.38 35.79)
-		(end 249.94 33.23)
+		(start 243.94 35.18)
+		(end 243.94 33.23)
 		(width 0.3)
 		(layer "F.Cu")
@@
 	)
 	(segment
-		(start 227.52 53.84)
-		(end 245.57 35.79)
+		(start 226.02 53.13)
+		(end 243.15 36)
 		(width 0.3)
 		(layer "F.Cu")
@@
 	)
 	(segment
-		(start 226.52 53.4)
-		(end 245.94 33.98)
+		(start 226.02 59.8836)
+		(end 226.02 53.13)
 		(width 0.3)
 		(layer "F.Cu")
-		(net 56)
+		(net 55)
 	)
 	(segment
-		(start 245.94 33.98)
-		(end 245.94 33.23)
+		(start 245.57 35.79)
+		(end 247.38 35.79)
 		(width 0.3)
 		(layer "F.Cu")
@@
 	)
 	(segment
-		(start 226.52 59.8836)
-		(end 226.52 53.4)
+		(start 227.52 59.8836)
+		(end 227.52 53.84)
 		(width 0.3)
 		(layer "F.Cu")
@@
 	)
 	(segment
-		(start 245.35 35.27)
-		(end 245.9 35.27)
+		(start 247.38 35.79)
+		(end 249.94 33.23)
 		(width 0.3)
 		(layer "F.Cu")
-		(net 57)
+		(net 56)
 	)
 	(segment
-		(start 245.9 35.27)
-		(end 247.94 33.23)
+		(start 227.52 53.84)
+		(end 245.57 35.79)
 		(width 0.3)
 		(layer "F.Cu")
-		(net 57)
+		(net 56)
 	)
 	(segment
-		(start 248.1 33.4)
-		(end 248.1 32.68)
+		(start 226.52 53.4)
+		(end 245.94 33.98)
 		(width 0.3)
 		(layer "F.Cu")
@@
 	)
 	(segment
-		(start 227.020001 53.599999)
-		(end 245.35 35.27)
+		(start 245.94 33.98)
+		(end 245.94 33.23)
 		(width 0.3)
 		(layer "F.Cu")
@@
 	)
 	(segment
-		(start 227.020001 59.8836)
-		(end 227.020001 53.599999)
+		(start 226.52 59.8836)
+		(end 226.52 53.4)
 		(width 0.3)
 		(layer "F.Cu")
@@
 	)
 	(segment
-		(start 243.15 36)
-		(end 243.15 35.97)
+		(start 245.35 35.27)
+		(end 245.9 35.27)
 		(width 0.3)
 		(layer "F.Cu")
@@
 	)
 	(segment
-		(start 243.15 35.97)
-		(end 243.94 35.18)
+		(start 245.9 35.27)
+		(end 247.94 33.23)
 		(width 0.3)
 		(layer "F.Cu")
@@
 	)
 	(segment
-		(start 243.94 35.18)
-		(end 243.94 33.23)
+		(start 248.1 33.4)
+		(end 248.1 32.68)
 		(width 0.3)
 		(layer "F.Cu")
@@
 	)
 	(segment
-		(start 226.02 53.13)
-		(end 243.15 36)
+		(start 227.020001 53.599999)
+		(end 245.35 35.27)
 		(width 0.3)
 		(layer "F.Cu")
@@
 	)
 	(segment
-		(start 226.02 59.8836)
-		(end 226.02 53.13)
+		(start 227.020001 59.8836)
+		(end 227.020001 53.599999)
 		(width 0.3)
 		(layer "F.Cu")
