File: pcb/SolarLoRaBox.kicad_pcb (KiCad board)
At the start: 4 copper layers, 71.3 x 92.8 mm, 57 parts, among them J1 Conn_01x02_Socket, J10 Conn_01x05_Socket, J2 Conn_01x02_Socket, J3 Conn_01x04_Socket, J4 Conn_ARM_SWD_TagConnect_TC2030, J5 Conn_01x04_Socket, J6 Conn_01x04_Socket, J7 Conn_01x04_Socket, J8 Conn_01x04_Socket, J9 Conn_01x04_Socket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

Commit message: pcb: non functional changes
Routing:
- net /RESET: track 97.7 -> 98.3 mm
- net GND: vias 389 -> 393
Other:
- board text added: "SolarLoRaBox 20250207 v0.0.2"
- board text removed: "SolarLoRaBox 20250121 v0.0.2"
Changed lines of the file:
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@@
 			(pintype "power_in")
 		)
+		(model "${KICAD8_3DMODEL_DIR}/Package_QFP.3dshapes/TQFP-48-1EP_7x7mm_P0.5mm_EP5x5mm.wrl"
+			(offset
+				(xyz 0 0 0)
+			)
+			(scale
+				(xyz 1 1 1)
+			)
+			(rotate
+				(xyz 0 0 0)
+			)
+		)
 	)
 	(footprint "Resistor_SMD:R_0805_2012Metric_Pad1.20x1.40mm_HandSolder"
@@
 		)
 	)
-	(gr_text "SolarLoRaBox\n20250121\nv0.0.2"
+	(gr_text "SolarLoRaBox\n20250207\nv0.0.2"
 		(at 219.65 94.48 0)
 		(layer "F.SilkS")
@@
 	)
 	(via
+		(at 212.48 42.77)
+		(size 0.5)
+		(drill 0.3)
+		(layers "F.Cu" "B.Cu")
+		(free yes)
+		(net 2)
+	)
+	(via
 		(at 222.720001 54.8664)
 		(size 0.5)
@@
 	)
 	(via
+		(at 191.95 39.71)
+		(size 0.5)
+		(drill 0.3)
+		(layers "F.Cu" "B.Cu")
+		(free yes)
+		(net 2)
+	)
+	(via
 		(at 188.34 91.47)
 		(size 0.5)
@@
 	)
 	(via
+		(at 234.93 59.48)
+		(size 0.5)
+		(drill 0.3)
+		(layers "F.Cu" "B.Cu")
+		(free yes)
+		(net 2)
+	)
+	(via
 		(at 234.07 114.36)
 		(size 0.5)
@@
 	)
 	(via
-		(at 233.68 59.3)
+		(at 228.1 78.95)
 		(size 0.5)
 		(drill 0.3)
@@
 	)
 	(via
-		(at 228.1 78.95)
+		(at 192.21 42.4)
 		(size 0.5)
 		(drill 0.3)
@@
 	)
 	(via
+		(at 233.94 60.43)
+		(size 0.5)
+		(drill 0.3)
+		(layers "F.Cu" "B.Cu")
+		(free yes)
+		(net 2)
+	)
+	(via
 		(at 209.68 56.57)
 		(size 0.5)
@@
 	)
 	(segment
+		(start 233.33 60.19)
+		(end 232.58 60.19)
+		(width 0.3)
+		(layer "F.Cu")
+		(net 4)
+	)
+	(segment
 		(start 230.4864 61.35)
 		(end 231.42 61.35)
@@
 	)
 	(segment
-		(start 233.9 60.19)
-		(end 234.405 59.685)
-		(width 0.3)
-		(layer "F.Cu")
-		(net 4)
-	)
-	(segment
 		(start 252.14 86.87)
 		(end 252.14 85.5375)
@@
 	)
 	(segment
-		(start 234.61 59.48)
-		(end 234.61 58.1575)
+		(start 234.06 59.46)
+		(end 234.61 58.91)
 		(width 0.3)
 		(layer "F.Cu")
@@
 	)
 	(segment
-		(start 234.405 59.685)
-		(end 234.61 59.48)
-		(width 0.3)
-		(layer "F.Cu")
-		(net 4)
-	)
-	(segment
 		(start 248.805 43.21)
 		(end 248.805 43.913908)
@@
 	)
 	(segment
-		(start 232.58 60.19)
-		(end 233.9 60.19)
+		(start 218.730001 54.8564)
+		(end 218.740001 54.8464)
 		(width 0.3)
 		(layer "F.Cu")
@@
 	)
 	(segment
-		(start 218.730001 54.8564)
-		(end 218.740001 54.8464)
+		(start 234.06 59.46)
+		(end 233.33 60.19)
 		(width 0.3)
 		(layer "F.Cu")
@@
 	)
 	(segment
+		(start 234.61 58.91)
+		(end 234.61 58.1575)
+		(width 0.3)
+		(layer "F.Cu")
+		(net 4)
+	)
+	(segment
 		(start 223.52 59.8836)
 		(end 223.52 58.653899)
@@
 	)
 	(via
-		(at 234.405 59.685)
+		(at 234.06 59.46)
 		(size 0.5)
 		(drill 0.3)
@@
 	)
 	(segment
-		(start 212.9464 56.8936)
-		(end 212.98 56.86)
+		(start 214.5864 57.8364)
+		(end 218.730001 57.8364)
 		(width 0.4)
 		(layer "F.Cu")
@@
 	)
 	(segment
-		(start 212.9464 57.8364)
-		(end 218.730001 57.8364)
+		(start 212.98 56.23)
+		(end 214.5864 57.8364)
 		(width 0.4)
 		(layer "F.Cu")
@@
 	)
 	(segment
-		(start 212.9464 57.8364)
-		(end 212.9464 56.8936)
+		(start 212.98 56.23)
+		(end 212.98 51.21)
 		(width 0.4)
 		(layer "F.Cu")
@@
 	)
 	(segment
-		(start 212.98 56.86)
-		(end 212.98 51.21)
-		(width 0.4)
-		(layer "F.Cu")
-		(net 7)
-	)
-	(segment
 		(start 218.73 58.94)
 		(end 218.730001 58.939999)
@@
 	)
 	(via
-		(at 212.9464 57.8364)
+		(at 212.98 56.23)
 		(size 0.5)
 		(drill 0.3)
@@
 	)
 	(segment
+		(start 212.98 57.8028)
+		(end 210.55 60.2328)
+		(width 0.4)
+		(layer "B.Cu")
+		(net 7)
+	)
+	(segment
+		(start 210.55 60.2328)
+		(end 210.55 76.84)
+		(width 0.4)
+		(layer "B.Cu")
+		(net 7)
+	)
+	(segment
 		(start 252.33 46.8)
 		(end 240.62 46.8)
@@
 	)
 	(segment
-		(start 212.9464 57.8364)
-		(end 210.55 60.2328)
-		(width 0.4)
-		(layer "B.Cu")
-		(net 7)
-	)
-	(segment
 		(start 223.5 64.35)
 		(end 225.38 64.35)
@@
 	)
 	(segment
-		(start 210.55 60.2328)
-		(end 210.55 76.84)
+		(start 212.98 56.23)
+		(end 212.98 57.8028)
 		(width 0.4)
 		(layer "B.Cu")
